Commit message: Modifications to MyzharBot configuration

File: myzharbot_robot.urdf (robot description, URDF)
Before this commit: robot myfirst, 3 links, 2 joints
Links:
- added link body_link; visual box size=0.27 .27 .055
- link Left_wheel: geometry visual cylinder length=.03 radius=0.034925
- link Right_wheel: geometry visual cylinder length=.03 radius=0.034925
- link base_link: geometry visual cylinder length=.03 radius=0.03
Joints:
- added joint Body: type continuous, parent base_link, child body_link, origin xyz=0 0 0.09 rpy=0 0 0, axis 0 0 1
- joint Left: origin xyz=0 0.069 -0.085 rpy=1.57075 0 0 -> xyz=0 0.135 0.135 rpy=1.57075 0 0
- joint Right: origin xyz=0 -0.069 -0.085 rpy=1.57075 0 0 -> xyz=0 -0.135 0.135 rpy=1.57075 0 0

Commit message: Added parameter "/info/robot_name"

File: myzharbot_robot.urdf (robot description, URDF)
Before this commit: robot myzharbot, 4 links, 3 joints
Links:
- removed link body_link
- added link body_chassis_link; visual box size=0.27 .27 .055
Joints:
- joint Body: child body_link -> body_chassis_link; origin xyz=0 0 0.09 rpy=0 0 0 -> xyz=0 0 0 rpy=0 0 0

Commit message: Updated URDF model and TF broadcaster

File: myzharbot_robot.urdf (robot description, URDF)
Before this commit: robot myzharbot, 4 links, 3 joints
Links:
- added link spr_bfl; visual cylinder length=.07 radius=0.047625
- added link spr_bfr; visual cylinder length=.07 radius=0.047625
- added link spr_brl; visual cylinder length=.07 radius=0.047625
- added link spr_brr; visual cylinder length=.07 radius=0.047625
- link base_link: geometry visual cylinder length=.01 radius=0.01
- link body_chassis_link: geometry visual box size=0.27 0.27 .055
Joints:
- added joint Sprocket_bfl: type continuous, parent base_link, child spr_bfl, origin xyz=0.0 0.0 0.0 rpy=0 0 0, axis 0 0 1, limit effort=100 velocity=100
- added joint Sprocket_bfr: type continuous, parent base_link, child spr_bfr, origin xyz=0.0 0.0 0.0 rpy=0 0 0, axis 0 0 1, limit effort=100 velocity=100
- added joint Sprocket_brl: type continuous, parent base_link, child spr_brl, origin xyz=0.0 0.0 0.0 rpy=0 0 0, axis 0 0 1, limit effort=100 velocity=100
- added joint Sprocket_brr: type continuous, parent base_link, child spr_brr, origin xyz=0.0 0.0 0.0 rpy=0 0 0, axis 0 0 1, limit effort=100 velocity=100
- joint Body: origin xyz=0 0 0 rpy=0 0 0 -> xyz=0 0 0.0775 rpy=0 0 0
- joint Left: origin xyz=0 0.135 0.135 rpy=1.57075 0 0 -> xyz=-0.055 0.150 0.150 rpy=1.57075 0 0
- joint Right: origin xyz=0 -0.135 0.135 rpy=1.57075 0 0 -> xyz=-0.055 -0.150 0.150 rpy=1.57075 0 0
