Commit message: first working model

File: urdf/active_sprocket.urdf.xacro (robot description, xacro)
@@ -1,3 +1,21 @@
 <?xml version="1.0"?>
 <robot xmlns:xacro="http://ros.org/wiki/xacro" name="myzharbot_active_sprocket">
+  <xacro:macro name="myzharbot_active_sprocket" params="position *joint_pose">
+    <link name="${position}_wheel">
+      <visual>
+        <geometry>
+          <cylinder length="${active_sprocket_leght}" radius="${active_sprocket_radius}"/>
+        </geometry>
+        <material name="DarkGrey" />
+      </visual>
+    </link>
+    <joint name="${position}" type="continuous">
+      <parent link="base_link"/>
+      <child link="${position}_wheel"/>
+      <limit effort="100" velocity="100"/>
+      <joint_properties damping="0.0" friction="0.0"/>
+      <xacro:insert_block name="joint_pose"/>
+      <axis xyz="0 0 1"/>
+    </joint>
+  </xacro:macro>
 </robot>

File: urdf/myzharbot.urdf.xacro (robot description, xacro)
@@ -14,20 +14,42 @@
   <property name="active_sprocket_leght" value="0.034925"/>
   <property name="passive_sprocket_leght" value="0.047625"/>
-  <property name="sprocket_offset_x" value="0.135"/>
-  <property name="sprocket_offset_y" value="0.170"/>
-  <property name="sprocket_offset_z" value="0.047625"/>
+  <property name="passive_sprocket_offset_x" value="0.135"/>
+  <property name="passive_sprocket_offset_y" value="0.170"/>
+  <property name="passive_sprocket_offset_z" value="0.047625"/>
+  <property name="active_sprocket_offset_x" value="0.055"/>
+  <property name="active_sprocket_offset_y" value="0.150"/>
+  <property name="active_sprocket_offset_z" value="0.150"/>
   <!-- Sprockets params -->
+  <!-- base_link -->
+  <link name="base_link">
+	<visual>
+	    <origin xyz="0 0 0" rpy="0 0 0" />
+            <geometry>
+                <cylinder length=".01" radius="0.1"/>
+            </geometry>
+            <material name="Red" />
+        </visual>
+  </link>
+  <!-- base_link -->
+  <!-- Active Sprockets -->
+  <xacro:myzharbot_active_sprocket position="Left">
+    <origin xyz="${active_sprocket_offset_x} ${-active_sprocket_offset_y} ${active_sprocket_offset_z}" rpy="${M_PI/2} 0 0" />
+  </xacro:myzharbot_active_sprocket>
+  <xacro:myzharbot_active_sprocket position="Right">
+    <origin xyz="${active_sprocket_offset_x} ${active_sprocket_offset_y} ${active_sprocket_offset_z}" rpy="${M_PI/2} 0 ${M_PI}" />
+  </xacro:myzharbot_active_sprocket>
+  <!-- Active Sprockets -->
   <!-- Passive Sprockets -->
   <xacro:myzharbot_passive_sprocket sprocket_suffix="bfl" position="Left">
-    <origin xyz="${sprocket_offset_x} ${sprocket_offset_y} ${wheel_vertical_offset}" rpy="0 0 0" />
+    <origin xyz="${passive_sprocket_offset_x} ${-passive_sprocket_offset_y} ${passive_sprocket_offset_z}" rpy="${M_PI/2} 0 0" />
   </xacro:myzharbot_passive_sprocket>
   <xacro:myzharbot_passive_sprocket sprocket_suffix="brl" position="Left">
-    <origin xyz="${sprocket_offset_x} -${sprocket_offset_y} ${sprocket_offset_z}" rpy="0 0 0" />
+    <origin xyz="${-passive_sprocket_offset_x} ${-passive_sprocket_offset_y} ${passive_sprocket_offset_z}" rpy="${M_PI/2} 0 0" />
   </xacro:myzharbot_passive_sprocket>
   <xacro:myzharbot_passive_sprocket sprocket_suffix="bfr" position="Right">
-    <origin xyz="-${sprocket_offset_x} ${sprocket_offset_y} ${sprocket_offset_z}" rpy="0 0 0" />
+    <origin xyz="${passive_sprocket_offset_x} ${passive_sprocket_offset_y} ${passive_sprocket_offset_z}" rpy="${M_PI/2} 0 ${M_PI}" />
   </xacro:myzharbot_passive_sprocket>
   <xacro:myzharbot_passive_sprocket sprocket_suffix="brr" position="Right">
-    <origin xyz="-${sprocket_offset_x} -${sprocket_offset_y} ${sprocket_offset_z}" rpy="0 0 0" />
+    <origin xyz="${-passive_sprocket_offset_x} ${passive_sprocket_offset_y} ${passive_sprocket_offset_z}" rpy="${M_PI/2} 0 ${M_PI}" />
   </xacro:myzharbot_passive_sprocket>
   <!-- Passive Sprockets -->

File: urdf/passive_sprocket.urdf.xacro (robot description, xacro)
@@ -1,32 +1,30 @@
 <?xml version="1.0"?>
 <robot xmlns:xacro="http://ros.org/wiki/xacro" name="myzharbot_passive_sprocket">
-  <xacro:macro name="myzharbot_passive_sprocket" params="sprocket_suffix active_sprocket_radius passive_sprocket_radius passive_sprocket_leght position">
+  <xacro:macro name="myzharbot_passive_sprocket" params="sprocket_suffix position *joint_pose">
     <link name="spr_${sprocket_suffix}">
       <visual>
         <geometry>
-          <cylinder length=${passive_sprocket_leght} radius=${passive_sprocket_radius}/>
+          <cylinder length="${passive_sprocket_leght}" radius="${passive_sprocket_radius}"/>
         </geometry>
-        <material name="dark_grey">
-          <color rgba="0.1 0.1 0.1 0.9"/>
-        </material>
+        <material name="DarkGrey" />
       </visual>
     </link>
     <joint name="Sprocket_${sprocket_suffix}" type="continuous">
-      <axis xyz="0 0 1"/>
       <parent link="base_link"/>
       <child link="spr_${sprocket_suffix}"/>
-      <origin rpy="0 0 0" xyz="0.0 0.0 0.0"/>
       <limit effort="100" velocity="100"/>
       <joint_properties damping="0.0" friction="0.0"/>
+      <xacro:insert_block name="joint_pose"/>
+      <axis xyz="0 0 1" rpy="0 0 0"/>
     </joint>
     <transmission name="sprocket_trans_${sprocket_suffix}" type="SimpleTransmission">
-  			<type>transmission_interface/SimpleTransmission</type>
-  			<actuator name="${position}_wheel">
-  				<mechanicalReduction>${active_sprocket_radius}/${passive_sprocket_radius}</mechanicalReduction>
-  			</actuator>
-  			<joint name="Sprocket_${sprocket_suffix}">
-  				<hardwareInterface>VelocityJointInterface</hardwareInterface>
-  			</joint>
-  		</transmission>
-	</xacro:macro>
+       <type>transmission_interface/SimpleTransmission</type>
+       <actuator name="${position}_wheel">
+          <mechanicalReduction>${active_sprocket_radius/passive_sprocket_radius}</mechanicalReduction>
+       </actuator>
+       <joint name="Sprocket_${sprocket_suffix}">
+          <hardwareInterface>VelocityJointInterface</hardwareInterface>
+       </joint>
+    </transmission>
+  </xacro:macro>
 </robot>
