Commit message: Passive Sprockets

File: urdf/myzharbot.urdf.xacro (robot description, xacro)
@@ -1,4 +1,28 @@
+<?xml version="1.0"?>
 <robot name="myzharbot_robot" xmlns:xacro="http://ros.org/wiki/xacro">
   <xacro:include filename="$(find myzharbot_description)/urdf/tracks.urdf.xacro" />
   <property name="M_PI" value="3.14159"/>
+  <!-- Sprockets params -->
+  <property name="active_sprocket_radius" value="0.034925"/>
+  <property name="passive_sprocket_radius" value="0.047625"/>
+  <property name="active_sprocket_leght" value="0.034925"/>
+  <property name="passive_sprocket_leght" value="0.047625"/>
+  <property name="sprocket_offset_x" value="0.135"/>
+  <property name="sprocket_offset_y" value="0.170"/>
+  <property name="sprocket_offset_z" value="0.047625"/>
+  <!-- Sprockets params -->
+  <!-- Passive Sprockets -->
+  <xacro:myzharbot_passive_sprocket sprocket_suffix="bfl" position="Left">
+    <origin xyz="${sprocket_offset_x} ${sprocket_offset_y} ${wheel_vertical_offset}" rpy="0 0 0" />
+  </xacro:myzharbot_passive_sprocket>
+  <xacro:myzharbot_passive_sprocket sprocket_suffix="brl" position="Left">
+    <origin xyz="${sprocket_offset_x} -${sprocket_offset_y} ${sprocket_offset_z}" rpy="0 0 0" />
+  </xacro:myzharbot_passive_sprocket>
+  <xacro:myzharbot_passive_sprocket sprocket_suffix="bfr" position="Right">
+    <origin xyz="-${sprocket_offset_x} ${sprocket_offset_y} ${sprocket_offset_z}" rpy="0 0 0" />
+  </xacro:myzharbot_passive_sprocket>
+  <xacro:myzharbot_passive_sprocket sprocket_suffix="brr" position="Right">
+    <origin xyz="-${sprocket_offset_x} -${sprocket_offset_y} ${sprocket_offset_z}" rpy="0 0 0" />
+  </xacro:myzharbot_passive_sprocket>
+  <!-- Passive Sprockets -->
 </robot>

Commit message: Added interactive marker twist server functionality  / Added useful launcher  / TODO change passive sprocket link and joint to dynamic and propagate joint transmission

File: urdf/myzharbot.urdf.xacro (robot description, xacro)
@@ -23,33 +23,49 @@
   <!-- base_link -->
   <link name="base_link">
-	<visual>
-	    <origin xyz="0 0 0" rpy="0 0 0" />
-            <geometry>
-                <cylinder length=".01" radius="0.1"/>
-            </geometry>
-            <material name="Red" />
-        </visual>
+    <visual>
+      <geometry>
+        <cylinder length=".01" radius="0.1"/>
+      </geometry>
+      <material name="Red" />
+    </visual>
   </link>
   <!-- base_link -->
+  <!-- Body chassis -->
+  <link name="body_chassis_link">
+    <visual>
+      <geometry>
+        <box size="0.27 0.27 .055"/>
+      </geometry>
+      <material name="Black" />
+    </visual>
+  </link>
+  <joint name="Body" type="fixed">
+    <axis xyz="0 0 1"/>
+    <parent link="base_link"/>
+    <child link="body_chassis_link"/>
+    <origin rpy="0 0 0" xyz="0 0 0.0775"/>
+    <joint_properties damping="0.0" friction="0.0"/>
+  </joint>
+  <!-- Body chassis -->
   <!-- Active Sprockets -->
   <xacro:myzharbot_active_sprocket position="Left">
-    <origin xyz="${active_sprocket_offset_x} ${-active_sprocket_offset_y} ${active_sprocket_offset_z}" rpy="${M_PI/2} 0 0" />
+    <origin xyz="${active_sprocket_offset_x} ${active_sprocket_offset_y} ${active_sprocket_offset_z}" rpy="${-M_PI/2} 0 0" />
   </xacro:myzharbot_active_sprocket>
   <xacro:myzharbot_active_sprocket position="Right">
-    <origin xyz="${active_sprocket_offset_x} ${active_sprocket_offset_y} ${active_sprocket_offset_z}" rpy="${M_PI/2} 0 ${M_PI}" />
+    <origin xyz="${active_sprocket_offset_x} ${-active_sprocket_offset_y} ${active_sprocket_offset_z}" rpy="${-M_PI/2} 0 0" />
   </xacro:myzharbot_active_sprocket>
   <!-- Active Sprockets -->
   <!-- Passive Sprockets -->
   <xacro:myzharbot_passive_sprocket sprocket_suffix="bfl" position="Left">
-    <origin xyz="${passive_sprocket_offset_x} ${-passive_sprocket_offset_y} ${passive_sprocket_offset_z}" rpy="${M_PI/2} 0 0" />
+    <origin xyz="${passive_sprocket_offset_x} ${passive_sprocket_offset_y} ${passive_sprocket_offset_z}" rpy="${-M_PI/2} 0 0" />
   </xacro:myzharbot_passive_sprocket>
   <xacro:myzharbot_passive_sprocket sprocket_suffix="brl" position="Left">
-    <origin xyz="${-passive_sprocket_offset_x} ${-passive_sprocket_offset_y} ${passive_sprocket_offset_z}" rpy="${M_PI/2} 0 0" />
+    <origin xyz="${-passive_sprocket_offset_x} ${passive_sprocket_offset_y} ${passive_sprocket_offset_z}" rpy="${-M_PI/2} 0 0" />
   </xacro:myzharbot_passive_sprocket>
   <xacro:myzharbot_passive_sprocket sprocket_suffix="bfr" position="Right">
-    <origin xyz="${passive_sprocket_offset_x} ${passive_sprocket_offset_y} ${passive_sprocket_offset_z}" rpy="${M_PI/2} 0 ${M_PI}" />
+    <origin xyz="${passive_sprocket_offset_x} ${-passive_sprocket_offset_y} ${passive_sprocket_offset_z}" rpy="${-M_PI/2} 0 0" />
   </xacro:myzharbot_passive_sprocket>
   <xacro:myzharbot_passive_sprocket sprocket_suffix="brr" position="Right">
-    <origin xyz="${-passive_sprocket_offset_x} ${passive_sprocket_offset_y} ${passive_sprocket_offset_z}" rpy="${M_PI/2} 0 ${M_PI}" />
+    <origin xyz="${-passive_sprocket_offset_x} ${-passive_sprocket_offset_y} ${passive_sprocket_offset_z}" rpy="${-M_PI/2} 0 0" />
   </xacro:myzharbot_passive_sprocket>
   <!-- Passive Sprockets -->

File: urdf/passive_sprocket.urdf.xacro (robot description, xacro)
@@ -10,5 +10,5 @@
       </visual>
     </link>
-    <joint name="Sprocket_${sprocket_suffix}" type="continuous">
+    <joint name="Sprocket_${sprocket_suffix}" type="fixed">
       <parent link="base_link"/>
       <child link="spr_${sprocket_suffix}"/>
@@ -20,5 +20,5 @@
     <transmission name="sprocket_trans_${sprocket_suffix}" type="SimpleTransmission">
        <type>transmission_interface/SimpleTransmission</type>
-       <actuator name="${position}_wheel">
+       <actuator name="${position}">
           <mechanicalReduction>${active_sprocket_radius/passive_sprocket_radius}</mechanicalReduction>
        </actuator>

Commit message: Added particulars to virtual model

File: urdf/myzharbot.urdf.xacro (robot description, xacro)
@@ -5,4 +5,5 @@
   <xacro:include filename="$(find myzharbot_robot_ros)/urdf/passive_sprocket.urdf.xacro" />
   <xacro:include filename="$(find myzharbot_robot_ros)/urdf/active_sprocket.urdf.xacro" />
+  <xacro:include filename="$(find myzharbot_robot_ros)/urdf/motor.urdf.xacro" />
   <xacro:include filename="$(find myzharbot_robot_ros)/urdf/sensors/asus_xtion_pro.urdf.xacro"/>
   <!-- Included URDF/XACRO Files -->
@@ -16,15 +17,23 @@
   <property name="passive_sprocket_leght" value="0.047625"/>
   <property name="passive_sprocket_offset_x" value="0.135"/>
-  <property name="passive_sprocket_offset_y" value="0.170"/>
+  <property name="passive_sprocket_offset_y" value="0.165"/>
   <property name="passive_sprocket_offset_z" value="0.047625"/>
   <property name="active_sprocket_offset_x" value="0.055"/>
-  <property name="active_sprocket_offset_y" value="0.150"/>
+  <property name="active_sprocket_offset_y" value="0.160"/>
   <property name="active_sprocket_offset_z" value="0.150"/>
   <!-- Sprockets params -->
+  <!-- Asus Xtion params -->
+  <property name="cam_px" value="-0.095" />
+  <property name="cam_py" value="-0.022" />
+  <property name="cam_pz" value="0.1825" />
+  <property name="cam_or" value="0" />
+  <property name="cam_op" value="0" />
+  <property name="cam_oy" value="${M_PI}" />
+  <!-- Asus Xtion params -->
   <!-- base_link -->
   <link name="base_link">
     <visual>
       <geometry>
-        <cylinder length=".01" radius="0.1"/>
+        <cylinder length=".001" radius="0.05"/>
       </geometry>
       <material name="Red" />
@@ -33,27 +42,68 @@
   <!-- base_link -->
   <!-- Body chassis -->
-  <link name="body_chassis_link">
+  <link name="body_bottom_chassis_link">
     <visual>
       <geometry>
-        <box size="0.27 0.27 .055"/>
+        <box size="0.27 0.27 .005"/>
       </geometry>
       <material name="Black" />
     </visual>
   </link>
-  <joint name="Body" type="fixed">
+  <joint name="Body_bottom" type="fixed">
     <axis xyz="0 0 1"/>
     <parent link="base_link"/>
-    <child link="body_chassis_link"/>
-    <origin rpy="0 0 0" xyz="0 0 0.0775"/>
+    <child link="body_bottom_chassis_link"/>
+    <origin rpy="0 0 0" xyz="0 0 ${passive_sprocket_offset_z+0.01}"/>
+    <joint_properties damping="0.0" friction="0.0"/>
+  </joint>
+  <link name="body_top_chassis_link">
+    <visual>
+      <geometry>
+        <box size="0.13 0.27 .055"/>
+      </geometry>
+      <material name="Black" />
+    </visual>
+  </link>
+  <joint name="Body_top" type="fixed">
+    <axis xyz="0 0 1"/>
+    <parent link="base_link"/>
+    <child link="body_top_chassis_link"/>
+    <origin rpy="0 0 0" xyz="0.035 0 ${passive_sprocket_offset_z+0.0375}"/>
+    <joint_properties damping="0.0" friction="0.0"/>
+  </joint>
+  <link name="asus_support_link">
+    <visual>
+      <geometry>
+        <box size="0.015 0.015 .015"/>
+      </geometry>
+      <material name="Black" />
+    </visual>
+  </link>
+  <joint name="Asus_support" type="fixed">
+    <axis xyz="0 0 1"/>
+    <parent link="base_link"/>
+    <child link="asus_support_link"/>
+    <origin rpy="0 0 0" xyz="${cam_px+0.01725} 0 0.1575"/>
     <joint_properties damping="0.0" friction="0.0"/>
   </joint>
   <!-- Body chassis -->
+  <!-- Jetson chassis -->
+  <link name="jetson_chassis_link">
+    <visual>
+      <geometry>
+        <box size="0.13 0.15 .095"/>
+      </geometry>
+      <material name="Black" />
+    </visual>
+  </link>
+  <joint name="Jetson" type="fixed">
+    <axis xyz="0 0 1"/>
+    <parent link="base_link"/>
+    <child link="jetson_chassis_link"/>
+    <origin rpy="0 0 0" xyz="-0.035 0 ${passive_sprocket_offset_z+0.0125+0.0475}"/>
+    <joint_properties damping="0.0" friction="0.0"/>
+  </joint>
+  <!-- Jetson chassis -->
   <!-- Asus Xtion Pro Live -->
-  <property name="cam_px" value="-0.085" />
-  <property name="cam_py" value="-0.022" />
-  <property name="cam_pz" value="0.18" />
-  <property name="cam_or" value="0" />
-  <property name="cam_op" value="0" />
-  <property name="cam_oy" value="${M_PI}" />
   <xacro:sensor_asus_xtion_pro parent="base_link"/>
   <!-- Asus Xtion Pro Live -->
@@ -65,4 +115,10 @@
     <origin xyz="${active_sprocket_offset_x} ${-active_sprocket_offset_y} ${active_sprocket_offset_z}" rpy="${-M_PI/2} 0 0" />
   </xacro:myzharbot_active_sprocket>
+  <xacro:myzharbot_motor position="Left">
+    <origin xyz="${active_sprocket_offset_x} ${active_sprocket_offset_y-2*active_sprocket_leght} ${active_sprocket_offset_z}" rpy="${-M_PI/2} 0 0" />
+  </xacro:myzharbot_motor>
+  <xacro:myzharbot_motor position="Right">
+    <origin xyz="${active_sprocket_offset_x} ${-(active_sprocket_offset_y-2*active_sprocket_leght)} ${active_sprocket_offset_z}" rpy="${-M_PI/2} 0 0" />
+  </xacro:myzharbot_motor>
   <!-- Active Sprockets -->
   <!-- Passive Sprockets -->

File: urdf/passive_sprocket.urdf.xacro (robot description, xacro)
@@ -18,12 +18,13 @@
       <axis xyz="0 0 1" rpy="0 0 0"/>
     </joint>
-    <transmission name="sprocket_trans_${sprocket_suffix}" type="SimpleTransmission">
-       <type>transmission_interface/SimpleTransmission</type>
-       <actuator name="${position}">
-          <mechanicalReduction>${active_sprocket_radius/passive_sprocket_radius}</mechanicalReduction>
-       </actuator>
-       <joint name="Sprocket_${sprocket_suffix}">
-          <hardwareInterface>VelocityJointInterface</hardwareInterface>
-       </joint>
+    <transmission name="sprocket_trans_${sprocket_suffix}">
+    	<type>transmission_interface/SimpleTransmission</type>
+    	<joint name="Sprocket_${sprocket_suffix}">
+      		<hardwareInterface>EffortJointInterface</hardwareInterface>
+    	</joint>
+    	<actuator name="${position}">
+		<hardwareInterface>EffortJointInterface</hardwareInterface>
+      			<mechanicalReduction>${active_sprocket_radius/passive_sprocket_radius}</mechanicalReduction>
+        </actuator>
     </transmission>
   </xacro:macro>

Commit message: Correct the inversion on X axis of the virtual model

File: urdf/myzharbot.urdf.xacro (robot description, xacro)
@@ -19,15 +19,15 @@
   <property name="passive_sprocket_offset_y" value="0.165"/>
   <property name="passive_sprocket_offset_z" value="0.047625"/>
-  <property name="active_sprocket_offset_x" value="0.055"/>
+  <property name="active_sprocket_offset_x" value="-0.055"/>
   <property name="active_sprocket_offset_y" value="0.160"/>
   <property name="active_sprocket_offset_z" value="0.150"/>
   <!-- Sprockets params -->
   <!-- Asus Xtion params -->
-  <property name="cam_px" value="-0.095" />
-  <property name="cam_py" value="-0.022" />
+  <property name="cam_px" value="0.095" />
+  <property name="cam_py" value="0.022" />
   <property name="cam_pz" value="0.1825" />
   <property name="cam_or" value="0" />
   <property name="cam_op" value="0" />
-  <property name="cam_oy" value="${M_PI}" />
+  <property name="cam_oy" value="0" />
   <!-- Asus Xtion params -->
   <!-- base_link -->
@@ -69,5 +69,5 @@
     <parent link="base_link"/>
     <child link="body_top_chassis_link"/>
-    <origin rpy="0 0 0" xyz="0.035 0 ${passive_sprocket_offset_z+0.0375}"/>
+    <origin rpy="0 0 0" xyz="-0.035 0 ${passive_sprocket_offset_z+0.0375}"/>
     <joint_properties damping="0.0" friction="0.0"/>
   </joint>
@@ -84,5 +84,5 @@
     <parent link="base_link"/>
     <child link="asus_support_link"/>
-    <origin rpy="0 0 0" xyz="${cam_px+0.01725} 0 0.1575"/>
+    <origin rpy="0 0 0" xyz="${cam_px-0.01725} 0 0.1575"/>
     <joint_properties damping="0.0" friction="0.0"/>
   </joint>
@@ -101,5 +101,5 @@
     <parent link="base_link"/>
     <child link="jetson_chassis_link"/>
-    <origin rpy="0 0 0" xyz="-0.035 0 ${passive_sprocket_offset_z+0.0125+0.0475}"/>
+    <origin rpy="0 0 0" xyz="0.035 0 ${passive_sprocket_offset_z+0.0125+0.0475}"/>
     <joint_properties damping="0.0" friction="0.0"/>
   </joint>

Commit message: File reorganization

File: urdf/myzharbot.urdf.xacro (robot description, xacro)
@@ -34,4 +34,5 @@
   <link name="base_link">
     <visual>
+      <origin rpy="0 0 0" xyz="0 0 0"/>
       <geometry>
         <cylinder length=".001" radius="0.05"/>
