Commit message: Update passive_sprocket.urdf.xacro

File: urdf/passive_sprocket.urdf.xacro (robot description, xacro)
@@ -1,3 +1,32 @@
 <?xml version="1.0"?>
-  <robot xmlns:xacro="http://ros.org/wiki/xacro" name="myzharbot_passive_sprocket">
+<robot xmlns:xacro="http://ros.org/wiki/xacro" name="myzharbot_passive_sprocket">
+  <xacro:macro name="myzharbot_passive_sprocket" params="sprocket_suffix active_sprocket_radius passive_sprocket_radius passive_sprocket_leght position">
+    <link name="spr_${sprocket_suffix}">
+      <visual>
+        <geometry>
+          <cylinder length=${passive_sprocket_leght} radius=${passive_sprocket_radius}/>
+        </geometry>
+        <material name="dark_grey">
+          <color rgba="0.1 0.1 0.1 0.9"/>
+        </material>
+      </visual>
+    </link>
+    <joint name="Sprocket_${sprocket_suffix}" type="continuous">
+      <axis xyz="0 0 1"/>
+      <parent link="base_link"/>
+      <child link="spr_${sprocket_suffix}"/>
+      <origin rpy="0 0 0" xyz="0.0 0.0 0.0"/>
+      <limit effort="100" velocity="100"/>
+      <joint_properties damping="0.0" friction="0.0"/>
+    </joint>
+    <transmission name="sprocket_trans_${sprocket_suffix}" type="SimpleTransmission">
+  			<type>transmission_interface/SimpleTransmission</type>
+  			<actuator name="${position}_wheel">
+  				<mechanicalReduction>${active_sprocket_radius}/${passive_sprocket_radius}</mechanicalReduction>
+  			</actuator>
+  			<joint name="Sprocket_${sprocket_suffix}">
+  				<hardwareInterface>VelocityJointInterface</hardwareInterface>
+  			</joint>
+  		</transmission>
+	</xacro:macro>
 </robot>

Commit message: Added mimic to passive sprockets

File: urdf/passive_sprocket.urdf.xacro (robot description, xacro)
@@ -10,5 +10,5 @@
       </visual>
     </link>
-    <joint name="Sprocket_${sprocket_suffix}" type="fixed">
+    <joint name="Sprocket_${sprocket_suffix}" type="continuous">
       <parent link="base_link"/>
       <child link="spr_${sprocket_suffix}"/>
@@ -17,6 +17,7 @@
       <xacro:insert_block name="joint_pose"/>
       <axis xyz="0 0 1" rpy="0 0 0"/>
+      <mimic joint="${position}" multiplier="${active_sprocket_radius/passive_sprocket_radius}" offset="0"/>
     </joint>
-    <transmission name="sprocket_trans_${sprocket_suffix}">
+    <!-- <transmission name="sprocket_trans_${sprocket_suffix}">
     	<type>transmission_interface/SimpleTransmission</type>
     	<joint name="Sprocket_${sprocket_suffix}">
@@ -27,5 +28,5 @@
       			<mechanicalReduction>${active_sprocket_radius/passive_sprocket_radius}</mechanicalReduction>
         </actuator>
-    </transmission>
+    </transmission> -->
   </xacro:macro>
 </robot>

Commit message: minor change

File: urdf/passive_sprocket.urdf.xacro (robot description, xacro)
@@ -17,16 +17,7 @@
       <xacro:insert_block name="joint_pose"/>
       <axis xyz="0 0 1" rpy="0 0 0"/>
+      <!-- Passive sprocket rotate automatically according to the status of the active one -->
       <mimic joint="${position}" multiplier="${active_sprocket_radius/passive_sprocket_radius}" offset="0"/>
     </joint>
-    <!-- <transmission name="sprocket_trans_${sprocket_suffix}">
-    	<type>transmission_interface/SimpleTransmission</type>
-    	<joint name="Sprocket_${sprocket_suffix}">
-      		<hardwareInterface>EffortJointInterface</hardwareInterface>
-    	</joint>
-    	<actuator name="${position}">
-		<hardwareInterface>EffortJointInterface</hardwareInterface>
-      			<mechanicalReduction>${active_sprocket_radius/passive_sprocket_radius}</mechanicalReduction>
-        </actuator>
-    </transmission> -->
   </xacro:macro>
 </robot>
