Commit message: Correction after package name changing

File: urdf/description.xacro (robot description, xacro)
@@ -1,5 +1,5 @@
 <?xml version="1.0"?>
 <robot name="myzharbot" xmlns:xacro="http://ros.org/wiki/xacro">
-  <xacro:include filename="$(find myzharbot_robot_ros)/urdf/myzharbot.urdf.xacro" />
+  <xacro:include filename="$(find ros_myzharbot_robot)/urdf/myzharbot.urdf.xacro" />
   <xacro:myzharbot_robot />
 </robot>

File: urdf/myzharbot.urdf.xacro (robot description, xacro)
@@ -2,9 +2,9 @@
 <robot name="myzharbot_robot" xmlns:xacro="http://ros.org/wiki/xacro">
   <!-- Included URDF/XACRO Files -->
-  <xacro:include filename="$(find myzharbot_robot_ros)/urdf/materials.urdf" />
-  <xacro:include filename="$(find myzharbot_robot_ros)/urdf/passive_sprocket.urdf.xacro" />
-  <xacro:include filename="$(find myzharbot_robot_ros)/urdf/active_sprocket.urdf.xacro" />
-  <xacro:include filename="$(find myzharbot_robot_ros)/urdf/motor.urdf.xacro" />
-  <xacro:include filename="$(find myzharbot_robot_ros)/urdf/sensors/asus_xtion_pro.urdf.xacro"/>
+  <xacro:include filename="$(find ros_myzharbot_robot)/urdf/materials.urdf" />
+  <xacro:include filename="$(find ros_myzharbot_robot)/urdf/passive_sprocket.urdf.xacro" />
+  <xacro:include filename="$(find ros_myzharbot_robot)/urdf/active_sprocket.urdf.xacro" />
+  <xacro:include filename="$(find ros_myzharbot_robot)/urdf/motor.urdf.xacro" />
+  <xacro:include filename="$(find ros_myzharbot_robot)/urdf/sensors/asus_xtion_pro.urdf.xacro"/>
   <!-- Included URDF/XACRO Files -->
   <!-- Global properties -->

File: urdf/sensors/asus_xtion_pro.urdf.xacro (robot description, xacro)
@@ -30,5 +30,5 @@
         <origin xyz="-0.01 0 0" rpy="${-M_PI/2} -${M_PI} ${-M_PI/2}"/>
         <geometry>
-          <mesh filename="package://myzharbot_robot_ros/meshes/sensors/asus_xtion_pro_live.dae" scale="${M_SCALE} ${M_SCALE} ${M_SCALE}"/>
+          <mesh filename="package://ros_myzharbot_robot/meshes/sensors/asus_xtion_pro_live.dae" scale="${M_SCALE} ${M_SCALE} ${M_SCALE}"/>
         </geometry>
       </visual>
