Commit message: Fixed namespaces

File: urdf/sensors/asus_xtion_pro.urdf.xacro (robot description, xacro)
@@ -7,24 +7,24 @@
   <!-- Parameterised in part by the values in turtlebot_properties.urdf.xacro -->
   <xacro:macro name="sensor_asus_xtion_pro" params="parent">
-    <joint name="camera_rgb_joint" type="fixed">
+    <joint name="rgbd_camera_rgb_joint" type="fixed">
       <origin xyz="${cam_px} ${cam_py} ${cam_pz}"
               rpy="${cam_or} ${cam_op} ${cam_oy}"/>
       <parent link="${parent}"/>
-      <child link="camera_rgb_frame" />
+      <child link="rgbd_camera_rgb_frame" />
     </joint>
-    <link name="camera_rgb_frame"/>
+    <link name="rgbd_camera_rgb_frame"/>
     <joint name="camera_rgb_optical_joint" type="fixed">
       <origin xyz="0 0 0" rpy="${-M_PI/2} 0 ${-M_PI/2}" />
-      <parent link="camera_rgb_frame" />
-      <child link="camera_rgb_optical_frame" />
+      <parent link="rgbd_camera_rgb_frame" />
+      <child link="rgbd_camera_rgb_optical_frame" />
     </joint>
-    <link name="camera_rgb_optical_frame"/>
-    <joint name="camera_joint" type="fixed">
+    <link name="rgbd_camera_rgb_optical_frame"/>
+    <joint name="rgbd_camera_joint" type="fixed">
       <origin xyz="0 ${asus_xtion_pro_cam_rel_rgb_py} 0"
               rpy="0 0 0"/>
-      <parent link="camera_rgb_frame"/>
-      <child link="camera_link"/>
+      <parent link="rgbd_camera_rgb_frame"/>
+      <child link="rgbd_camera_link"/>
     </joint>
-    <link name="camera_link">
+    <link name="rgbd_camera_link">
       <visual>
         <origin xyz="-0.01 0 0" rpy="${-M_PI/2} -${M_PI} ${-M_PI/2}"/>
@@ -47,16 +47,16 @@
       </inertial>
     </link>
-    <joint name="camera_depth_joint" type="fixed">
+    <joint name="rgbd_camera_depth_joint" type="fixed">
       <origin xyz="0 ${asus_xtion_pro_depth_rel_rgb_py} 0" rpy="0 0 0" />
-      <parent link="camera_rgb_frame" />
-      <child link="camera_depth_frame" />
+      <parent link="rgbd_camera_rgb_frame" />
+      <child link="rgbd_camera_depth_frame" />
     </joint>
-    <link name="camera_depth_frame"/>
+    <link name="rgbd_camera_depth_frame"/>
     <joint name="camera_depth_optical_joint" type="fixed">
       <origin xyz="0 0 0" rpy="${-M_PI/2} 0 ${-M_PI/2}" />
-      <parent link="camera_depth_frame" />
-      <child link="camera_depth_optical_frame" />
+      <parent link="rgbd_camera_depth_frame" />
+      <child link="rgbd_camera_depth_optical_frame" />
     </joint>
-    <link name="camera_depth_optical_frame"/>
+    <link name="rgbd_camera_depth_optical_frame"/>
   </xacro:macro>
 </robot>
