Commit message: New configuration to use ROS-Control

File: myzharbot_description/urdf/active_sprocket.urdf.xacro (robot description, xacro)
@@ -9,4 +9,10 @@
         <material name="DarkGrey" />
       </visual>
+      <collision>
+        <origin xyz="0 0 0" rpy="0 0 0" />
+        <geometry>
+          <cylinder length="${active_sprocket_leght}" radius="${active_sprocket_radius}"/>
+        </geometry>
+      </collision>
     </link>
     <joint name="${position}" type="continuous">

File: myzharbot_description/urdf/description.xacro (robot description, xacro)
@@ -1,5 +1,5 @@
 <?xml version="1.0"?>
 <robot name="myzharbot" xmlns:xacro="http://ros.org/wiki/xacro">
-  <xacro:include filename="$(find ros_myzharbot_robot)/urdf/myzharbot.urdf.xacro" />
+  <xacro:include filename="$(find myzharbot_description)/urdf/myzharbot.urdf.xacro" />
   <xacro:myzharbot_robot />
 </robot>

File: myzharbot_description/urdf/myzharbot.urdf.xacro (robot description, xacro)
@@ -2,9 +2,9 @@
 <robot name="myzharbot_robot" xmlns:xacro="http://ros.org/wiki/xacro">
   <!-- Included URDF/XACRO Files -->
-  <xacro:include filename="$(find ros_myzharbot_robot)/urdf/materials.urdf" />
-  <xacro:include filename="$(find ros_myzharbot_robot)/urdf/passive_sprocket.urdf.xacro" />
-  <xacro:include filename="$(find ros_myzharbot_robot)/urdf/active_sprocket.urdf.xacro" />
-  <xacro:include filename="$(find ros_myzharbot_robot)/urdf/motor.urdf.xacro" />
-  <xacro:include filename="$(find ros_myzharbot_robot)/urdf/sensors/asus_xtion_pro.urdf.xacro"/>
+  <xacro:include filename="$(find myzharbot_description)/urdf/materials.urdf" />
+  <xacro:include filename="$(find myzharbot_description)/urdf/passive_sprocket.urdf.xacro" />
+  <xacro:include filename="$(find myzharbot_description)/urdf/active_sprocket.urdf.xacro" />
+  <xacro:include filename="$(find myzharbot_description)/urdf/motor.urdf.xacro" />
+  <xacro:include filename="$(find myzharbot_description)/urdf/sensors/asus_xtion_pro.urdf.xacro"/>
   <!-- Included URDF/XACRO Files -->
   <!-- Global properties -->
